File: kicadProject/lab6PCB.kicad_sch (KiCad schematic)
At the start: 13 parts, among them J1 Conn_01x08, J2 Conn_01x08

Commit message: Finished Gerber Files Organized
Parts:
- D1, D2, D3, D4, D5: footprint (none) -> LED_SMD:LED_0805_2012Metric_Pad1.15x1.40mm_HandSolder
- J1, J2: footprint (none) -> Connector_PinHeader_2.54mm:PinHeader_1x08_P2.54mm_Vertical
- R1, R2, R3, R4, R5: footprint (none) -> Resistor_SMD:R_0805_2012Metric_Pad1.20x1.40mm_HandSolder
- U1: footprint (none) -> Package_SO:DS1722_SOIC_8_Custom
